Commit message: 3d curve interpolation

File: urdf/sassa-robot/robot.urdf (robot description, URDF)
Before this commit: robot sassa, 23 links, 22 joints
Links:
- link arm2_sasm: mass 0.60856194490192350166 -> 0.60856194490192339064
- link arm3_sasm: mass 0.11356194490192343671 -> 0.11356194490192342283
- link helbow_sasm: mass 0.76500000000000001332 -> 0.76500000000000012434
- link helbow_sasm_2: mass 0.76500000000000001332 -> 0.76500000000000012434
- link helbow_sasm_3: mass 0.76500000000000001332 -> 0.76500000000000012434
- link helbow_sasm_4: mass 0.76500000000000001332 -> 0.76500000000000012434
- link lowerleg_sasm_2: mass 0.13199999999999997846 -> 0.13200000000000000622
- link lowerleg_sasm_3: mass 0.13199999999999997846 -> 0.13200000000000000622
- link lowerleg_sasm_4: mass 0.13199999999999997846 -> 0.13200000000000000622
- link upperleg_sasm: mass 0.8920000000000000151 -> 0.89200000000000012612
- link upperleg_sasm_2: mass 0.8920000000000000151 -> 0.89200000000000012612
- link upperleg_sasm_3: mass 0.8920000000000000151 -> 0.89200000000000012612
- link upperleg_sasm_4: mass 0.8920000000000000151 -> 0.89200000000000012612

Commit message: scenario1 WIP

File: urdf/sassa-robot/robot.urdf (robot description, URDF)
Before this commit: robot sassa, 23 links, 22 joints
Links:
- removed link gripper_2
- removed link ot_sasm
- added link end_effector_sasm, mass 0.10999999999999998668; collision mesh filename=package:///2408.stl; collision mesh filename=package:///end_effector.stl
- link arm2_sasm: mass 0.60856194490192339064 -> 0.60856194490192350166
- link arm3_sasm: mass 0.11356194490192342283 -> 0.11356194490192343671
- link gripper: mass 0.010000000000000000208 -> 0
- link upperleg_sasm: mass 0.89200000000000012612 -> 0.8920000000000000151
Joints:
- removed joint GripperLeft
- removed joint GripperRight
- added joint Gripper: type revolute, parent end_effector_sasm, child gripper, origin xyz=0.035000000000000086597 -0.012000000000000010658 0.025000000000000022204 rpy=3.141592653589793116 -3.5728716727440510907e-16 1.3877787807815824936e-16, axis 0 0 1, limit lower=0 upper=1.0471975511965976313 effort=9 velocity=20
- joint OT: child ot_sasm -> end_effector_sasm
