Commit message: Add 3 scenarios, pick and place, look over a table, move a box

File: urdf/objects/box1.urdf (robot description, URDF)
Before this commit: robot box, 1 links, 0 joints
Links:
- link box: geometry collision box size=.15 .3 .3; visual box size=.15 .3 .3

File: urdf/sassa-robot/robot.urdf (robot description, URDF)
Before this commit: robot sassa, 22 links, 21 joints
Links:
- link body_sasm: mass 3.4790000000000000924 -> 3.4790000000000009805
- link end_effector_sasm: mass 0.10999999999999998668 -> 0.11000000000000001443
- link helbow_sasm: mass 0.76500000000000012434 -> 0.76500000000000001332
- link helbow_sasm_2: mass 0.76500000000000012434 -> 0.76500000000000001332
- link helbow_sasm_3: mass 0.76500000000000012434 -> 0.76500000000000001332
- link helbow_sasm_4: mass 0.76500000000000012434 -> 0.76500000000000001332
- link lowerleg_sasm: mass 0.13200000000000000622 -> 0.13200000000000003397
- link lowerleg_sasm_2: mass 0.13200000000000000622 -> 0.13200000000000003397
- link lowerleg_sasm_3: mass 0.13200000000000000622 -> 0.13200000000000003397
- link lowerleg_sasm_4: mass 0.13200000000000000622 -> 0.13200000000000003397
- link upperleg_sasm_2: mass 0.89200000000000012612 -> 0.8920000000000000151
- link upperleg_sasm_3: mass 0.89200000000000012612 -> 0.8920000000000000151
Joints:
- joint Gripper: origin xyz=0.035000000000000086597 -0.012000000000000010658 0.025000000000000022204 rpy=3.141592653589793116 -3.5728716727440510907e-16 1.3877787807815824936e-16 -> xyz=0.034999999999999975575 -0.01199999999999999678 0.024999999999999994449 rpy=3.141592653589793116 -3.5728716727440510907e-16 1.3877787807815824936e-16
- joint OT: origin xyz=0.12000000000000032863 1.3877787807814456755e-17 -0.015000000000000082712 rpy=4.2353752921601641395e-31 1.1237174519383729543e-16 -1.3339013638364774884e-15 -> xyz=0.11999999999999994005 1.3877787807814456755e-17 -0.01500000000000000118 rpy=4.2353752921601641395e-31 1.1237174519383729543e-16 -1.3339013638364774884e-15
- joint arm3: origin xyz=0.084852813742387400708 -0.084852813742386845597 1.6897430194022276028e-15 rpy=4.2353752921601877865e-31 8.995699258773243279e-31 -0.785398163397448279 -> xyz=0.084852813742385513329 -0.084852813742385235773 2.2389905509276539029e-15 rpy=4.2353752921601877865e-31 8.995699258773243279e-31 -0.785398163397448279
