Commit message: URDF file generation and trajectory

File: urdf/sassa-robot-short-arm/robot_temp.urdf (robot description, URDF)
Before this commit: robot sassa-short-arm, 22 links, 21 joints
Links:
- link arm1_sasm: geometry collision mesh filename=package:///5015.stl; visual mesh filename=package:///5015.stl
- link arm2_sasm: geometry collision mesh filename=package:///5015.stl; collision mesh filename=package:///7015.stl
- link arm3_sasm: geometry collision mesh filename=package:///link.stl; visual mesh filename=package:///link.stl
- link body_sasm: geometry collision mesh filename=package:///body.stl; collision mesh filename=package:///body_panel.stl
- link end_effector_sasm: geometry collision mesh filename=package:///2408.stl; collision mesh filename=package:///end_effector.stl
- link gripper: geometry collision mesh filename=package:///gripper.stl; visual mesh filename=package:///gripper.stl
- link helbow_sasm: geometry collision mesh filename=package:///angle_motor_connect.stl; collision mesh filename=package:///rmdx8v3.stl
- link helbow_sasm_2: geometry collision mesh filename=package:///angle_motor_connect.stl; collision mesh filename=package:///rmdx8v3.stl
- link helbow_sasm_3: geometry collision mesh filename=package:///angle_motor_connect.stl; collision mesh filename=package:///rmdx8v3.stl
- link helbow_sasm_4: geometry collision mesh filename=package:///angle_motor_connect.stl; collision mesh filename=package:///rmdx8v3.stl
- link lowerleg_sasm: geometry collision mesh filename=package:///61804-2rs.stl; collision mesh filename=package:///61804-2rs.stl
- link lowerleg_sasm_2: geometry collision mesh filename=package:///61804-2rs.stl; collision mesh filename=package:///61804-2rs.stl
- link lowerleg_sasm_3: geometry collision mesh filename=package:///61804-2rs.stl; collision mesh filename=package:///61804-2rs.stl
- link lowerleg_sasm_4: geometry collision mesh filename=package:///61804-2rs.stl; collision mesh filename=package:///61804-2rs.stl
- link upperleg_sasm: geometry collision mesh filename=package:///61804-2rs.stl; collision mesh filename=package:///inline_connect.stl
- link upperleg_sasm_2: geometry collision mesh filename=package:///61804-2rs.stl; collision mesh filename=package:///inline_connect.stl
- link upperleg_sasm_3: geometry collision mesh filename=package:///61804-2rs.stl; collision mesh filename=package:///inline_connect.stl
- link upperleg_sasm_4: geometry collision mesh filename=package:///61804-2rs.stl; collision mesh filename=package:///inline_connect.stl
