Commit message: Trajectory and debug CLIK

File: urdf/sassa-robot-short-arm/robot.urdf (robot description, URDF)
Before this commit: robot sassa-short-arm, 22 links, 21 joints
Links:
- link body_sasm: mass 3.4789999999999992042 -> 3.4790000000000000924
- link end_effector_sasm: mass 0.10999999999999998668 -> 0.11000000000000000056
- link helbow_sasm: mass 0.76499999999999979128 -> 0.76500000000000001332
- link helbow_sasm_2: mass 0.76499999999999979128 -> 0.76500000000000001332
- link helbow_sasm_3: mass 0.76499999999999979128 -> 0.76500000000000001332
- link helbow_sasm_4: mass 0.76499999999999979128 -> 0.76500000000000001332
- link lowerleg_sasm: mass 0.13200000000000000622 -> 0.13200000000000003397
- link upperleg_sasm: mass 0.89199999999999979305 -> 0.8920000000000000151
- link upperleg_sasm_2: mass 0.89199999999999979305 -> 0.8920000000000000151
- link upperleg_sasm_3: mass 0.89199999999999979305 -> 0.8920000000000000151
- link upperleg_sasm_4: mass 0.89199999999999990408 -> 0.89200000000000012612

Commit message: adding CoM visualization in Gepetto Viewer and 3D trajectory

File: urdf/sassa-robot-short-arm/robot.urdf (robot description, URDF)
Before this commit: robot sassa-short-arm, 22 links, 21 joints
Links:
- link arm2_sasm: mass 0.56808517537055802649 -> 0.55458517537055795898
- link arm3_sasm: mass 0.073085175370557989294 -> 0.059585175370557984242
- link body_sasm: mass 3.4790000000000000924 -> 3.4789999999999987601
- link end_effector_sasm: mass 0.11000000000000000056 -> 0.10999999999999998668
- link helbow_sasm: mass 0.76500000000000001332 -> 0.7649999999999999023
- link helbow_sasm_2: mass 0.76500000000000001332 -> 0.7649999999999999023
- link helbow_sasm_3: mass 0.76500000000000001332 -> 0.7649999999999999023
- link helbow_sasm_4: mass 0.76500000000000001332 -> 0.7649999999999999023
- link lowerleg_sasm_2: mass 0.13200000000000000622 -> 0.13200000000000003397
- link lowerleg_sasm_3: mass 0.13200000000000000622 -> 0.13200000000000003397
- link lowerleg_sasm_4: mass 0.13200000000000000622 -> 0.13200000000000003397
- link upperleg_sasm: mass 0.8920000000000000151 -> 0.89199999999999990408
- link upperleg_sasm_2: mass 0.8920000000000000151 -> 0.89199999999999990408
- link upperleg_sasm_3: mass 0.8920000000000000151 -> 0.89199999999999990408
- link upperleg_sasm_4: mass 0.89200000000000012612 -> 0.89199999999999990408
Joints:
- joint Gripper: origin xyz=0.034999999999999920064 -0.01199999999999999678 0.024999999999999994449 rpy=3.141592653589793116 -3.5728716727440510907e-16 1.3877787807815824936e-16 -> xyz=0.034999999999999920064 -0.01199999999999999678 0.025000000000000001388 rpy=3.141592653589793116 -3.5728716727440510907e-16 1.3877787807815824936e-16
- joint OT: origin xyz=0.079999999999999960032 1.3877787807814456755e-17 -0.014999999999999999445 rpy=4.2353752921601641395e-31 1.1237174519383729543e-16 -1.3339013638364774884e-15 -> xyz=0.060000000000000053291 1.3877787807814456755e-17 -0.01499999999999999771 rpy=4.2353752921601641395e-31 1.1237174519383729543e-16 -1.3339013638364774884e-15
- joint arm3: origin xyz=0.056568542494923657049 -0.056568542494923268471 2.2397479442724408186e-15 rpy=4.2353752921601877865e-31 8.995699258773243279e-31 -0.785398163397448279 -> xyz=0.042426406871192701153 -0.042426406871192368087 2.2401266409448350653e-15 rpy=4.2353752921601877865e-31 8.995699258773243279e-31 -0.785398163397448279

File: urdf/sassa-robot/robot.urdf (robot description, URDF)
Before this commit: robot sassa, 22 links, 21 joints
Links:
- link arm1_sasm: geometry collision mesh filename=package:///5015.obj; visual mesh filename=package:///5015.obj
- link arm2_sasm: mass 0.60856194490192350166 -> 0.59508517537055793944; geometry collision mesh filename=package:///5015.obj; collision mesh filename=package:///7015.obj
- link arm3_sasm: mass 0.11356194490192343671 -> 0.1000851753705579994; geometry collision mesh filename=package:///link.obj; visual mesh filename=package:///link.obj
- link body_sasm: mass 3.4790000000000009805 -> 3.4789999999999992042; geometry collision mesh filename=package:///body.obj; collision mesh filename=package:///body_panel.obj
- link end_effector_sasm: mass 0.11000000000000001443 -> 0.10999999999999998668; geometry collision mesh filename=package:///2408.obj; collision mesh filename=package:///end_effector.obj
- link gripper: geometry collision mesh filename=package:///gripper.obj; visual mesh filename=package:///gripper.obj
- link helbow_sasm: mass 0.76500000000000001332 -> 0.76499999999999979128; geometry collision mesh filename=package:///angle_motor_connect.obj; collision mesh filename=package:///rmdx8v3.obj
- link helbow_sasm_2: mass 0.76500000000000001332 -> 0.76499999999999979128; geometry collision mesh filename=package:///angle_motor_connect.obj; collision mesh filename=package:///rmdx8v3.obj
- link helbow_sasm_3: mass 0.76500000000000001332 -> 0.76499999999999979128; geometry collision mesh filename=package:///angle_motor_connect.obj; collision mesh filename=package:///rmdx8v3.obj
- link helbow_sasm_4: mass 0.76500000000000001332 -> 0.76499999999999979128; geometry collision mesh filename=package:///angle_motor_connect.obj; collision mesh filename=package:///rmdx8v3.obj
- link lowerleg_sasm: mass 0.13200000000000003397 -> 0.13200000000000000622; geometry collision mesh filename=package:///61804-2rs.obj; collision mesh filename=package:///61804-2rs.obj
- link lowerleg_sasm_2: mass 0.13200000000000003397 -> 0.13200000000000000622; geometry collision mesh filename=package:///61804-2rs.obj; collision mesh filename=package:///61804-2rs.obj
- link lowerleg_sasm_3: mass 0.13200000000000003397 -> 0.13200000000000000622; geometry collision mesh filename=package:///61804-2rs.obj; collision mesh filename=package:///61804-2rs.obj
- link lowerleg_sasm_4: mass 0.13200000000000003397 -> 0.13200000000000000622; geometry collision mesh filename=package:///61804-2rs.obj; collision mesh filename=package:///61804-2rs.obj
- link upperleg_sasm: mass 0.8920000000000000151 -> 0.89199999999999990408; geometry collision mesh filename=package:///61804-2rs.obj; collision mesh filename=package:///inline_connect.obj
- link upperleg_sasm_2: mass 0.8920000000000000151 -> 0.89199999999999990408; geometry collision mesh filename=package:///61804-2rs.obj; collision mesh filename=package:///inline_connect.obj
- link upperleg_sasm_3: mass 0.8920000000000000151 -> 0.89199999999999990408; geometry collision mesh filename=package:///61804-2rs.obj; collision mesh filename=package:///inline_connect.obj
- link upperleg_sasm_4: mass 0.89200000000000012612 -> 0.89199999999999990408; geometry collision mesh filename=package:///61804-2rs.obj; collision mesh filename=package:///inline_connect.obj

Commit message: fixing mesh bad shading

File: urdf/sassa-robot-short-arm/robot.urdf (robot description, URDF)
Before this commit: robot sassa-short-arm, 22 links, 21 joints
Links:
- link arm2_sasm: mass 0.55458517537055795898 -> 0.56808517537055802649
- link arm3_sasm: mass 0.059585175370557984242 -> 0.073085175370557989294
- link body_sasm: mass 3.4789999999999987601 -> 3.4789999999999996483
- link end_effector_sasm: mass 0.10999999999999998668 -> 0.11000000000000001443
- link lowerleg_sasm_2: mass 0.13200000000000003397 -> 0.13200000000000000622
- link lowerleg_sasm_3: mass 0.13200000000000003397 -> 0.13200000000000000622
- link lowerleg_sasm_4: mass 0.13200000000000003397 -> 0.13200000000000000622
- link upperleg_sasm_4: mass 0.89199999999999990408 -> 0.8920000000000000151
Joints:
- joint Gripper: origin xyz=0.034999999999999920064 -0.01199999999999999678 0.025000000000000001388 rpy=3.141592653589793116 -3.5728716727440510907e-16 1.3877787807815824936e-16 -> xyz=0.034999999999999864553 -0.01199999999999999678 0.025000000000000001388 rpy=3.141592653589793116 -3.5728716727440510907e-16 1.3877787807815824936e-16
- joint OT: origin xyz=0.060000000000000053291 1.3877787807814456755e-17 -0.01499999999999999771 rpy=4.2353752921601641395e-31 1.1237174519383729543e-16 -1.3339013638364774884e-15 -> xyz=0.079999999999999960032 1.3877787807814456755e-17 -0.014999999999999999445 rpy=4.2353752921601641395e-31 1.1237174519383729543e-16 -1.3339013638364774884e-15
- joint arm3: origin xyz=0.042426406871192701153 -0.042426406871192368087 2.2401266409448350653e-15 rpy=4.2353752921601877865e-31 8.995699258773243279e-31 -0.785398163397448279 -> xyz=0.056568542494923657049 -0.056568542494923268471 2.2397479442724408186e-15 rpy=4.2353752921601877865e-31 8.995699258773243279e-31 -0.785398163397448279

File: urdf/sassa-robot/robot.urdf (robot description, URDF)
Before this commit: robot sassa, 22 links, 21 joints
Links:
- link body_sasm: mass 3.4789999999999992042 -> 3.4790000000000000924
- link end_effector_sasm: mass 0.10999999999999998668 -> 0.11000000000000000056
- link helbow_sasm: mass 0.76499999999999979128 -> 0.76500000000000012434
- link helbow_sasm_2: mass 0.76499999999999979128 -> 0.76500000000000012434
- link helbow_sasm_3: mass 0.76499999999999979128 -> 0.76500000000000012434
- link helbow_sasm_4: mass 0.76499999999999979128 -> 0.76500000000000012434
- link lowerleg_sasm: mass 0.13200000000000000622 -> 0.13200000000000003397
- link lowerleg_sasm_2: mass 0.13200000000000000622 -> 0.13200000000000003397
- link lowerleg_sasm_3: mass 0.13200000000000000622 -> 0.13200000000000003397
- link lowerleg_sasm_4: mass 0.13200000000000000622 -> 0.13200000000000003397
- link upperleg_sasm_2: mass 0.89199999999999990408 -> 0.8920000000000000151
- link upperleg_sasm_3: mass 0.89199999999999990408 -> 0.8920000000000000151
- link upperleg_sasm_4: mass 0.89199999999999990408 -> 0.89200000000000012612
Joints:
- joint Gripper: origin xyz=0.034999999999999975575 -0.01199999999999999678 0.024999999999999994449 rpy=3.141592653589793116 -3.5728716727440510907e-16 1.3877787807815824936e-16 -> xyz=0.034999999999999975575 -0.01199999999999999678 0.025000000000000001388 rpy=3.141592653589793116 -3.5728716727440510907e-16 1.3877787807815824936e-16
